Commit message: Fix size of collision box

File: urdf/tag_box.urdf.xacro (robot description, xacro)
@@ -18,5 +18,5 @@
       <origin xyz="0 0 0.15"/>
       <geometry>
-        <box size="0.3 0.3 0.3" />
+        <box size="0.2 0.2 0.2" />
       </geometry>
     </collision>

Commit message: Add parameterized mass,x,y,z & macro for inertia matrix

File: urdf/tag_box.urdf.xacro (robot description, xacro)
@@ -2,21 +2,31 @@
 <robot name="tag_box" xmlns:xacro="http://www.ros.org/wiki/xacro">
 <!-- This is for loading a box with one main link and different tags on each side -->
+<xacro:property name="mass" value="1.0" />
+<xacro:property name="x" value="0.2" />
+<xacro:property name="y" value="0.2" />
+<xacro:property name="z" value="0.2" />
+<!-- Macro for the inertia of a box -->
+<xacro:macro name="box_inertia" params="x y z mass">
+  <inertia ixx="${0.0833333 * mass * (y*y + z*z)}" ixy="0.0" ixz="0.0"
+  iyy="${0.0833333 * mass * (x*x + z*z)}" iyz="0.0"
+  izz="${0.0833333 * mass * (x*x + y*y)}" />
+</xacro:macro>
   <link name="tag_link">
     <inertial>
-      <origin xyz="0 0 0.15" />
-      <mass value="0.3" />
-      <inertia  ixx="1.0" ixy="0.0"  ixz="0.0"  iyy="1.0"  iyz="0.0"  izz="1.0" />
+      <origin xyz="0 0 0.1" />
+      <mass value="${mass}" />
+        <xacro:box_inertia x="${x}" y="${y}" z="${z}" mass="${mass}" />
     </inertial>
     <visual>
-      <origin xyz="0 0 0.15"/>
+      <origin xyz="0 0 0.1"/>
       <geometry>
-        <!-- AR Track Alvar -->
+        <!-- Mesh with AR Track Alvar tags -->
         <mesh filename="package://sortation_system/models/alvartags/meshes/alvartags$(arg tag_num).dae" />
       </geometry>
     </visual>
     <collision>
-      <origin xyz="0 0 0.15"/>
+      <origin xyz="0 0 0.1"/>
       <geometry>
-        <box size="0.2 0.2 0.2" />
+        <box size="${x} ${y} ${z}" />
       </geometry>
     </collision>
