Commit message: Add first cardboard boxes with a AR Tag on top

File: urdf/tag_box_0.urdf (robot description, URDF)
Before this commit: robot tag_box_0, 1 links, 0 joints
Links:
- removed link tag_link
- added link ar_tag; visual box size=0.1 0.1 0.0001
- added link box_link, mass 1.0; collision box size=0.515 0.356 0.2; visual mesh filename=package://sortation_system/media/meshes/cardboard_box.dae scale=1.3 0.9 0.5
Joints:
- added joint box_to_tag: type fixed, parent box_link, child ar_tag, origin xyz=0.0 0.0 0.3

File: urdf/tag_box_1.urdf (robot description, URDF)
Before this commit: robot tag_box_1, 1 links, 0 joints
Links:
- removed link tag_link
- added link ar_tag; visual box size=0.1 0.1 0.0001
- added link box_link, mass 1.0; collision box size=0.515 0.356 0.2; visual mesh filename=package://sortation_system/media/meshes/cardboard_box.dae scale=1.3 0.9 0.5
Joints:
- added joint box_to_tag: type fixed, parent box_link, child ar_tag, origin xyz=0.0 0.0 0.3
